Commit message: add parameters to the update rates for camera

File: urdf/_d435.gazebo.xacro (robot description, xacro)
@@ -6,5 +6,5 @@
 -->
 <robot xmlns:xacro="http://ros.org/wiki/xacro">
-  <xacro:macro name="gazebo_d435" params="camera_name reference_link topics_ns depth_optical_frame color_optical_frame infrared1_optical_frame infrared2_optical_frame publish_pointcloud:=true" >
+  <xacro:macro name="gazebo_d435" params="camera_name reference_link topics_ns depth_optical_frame color_optical_frame infrared1_optical_frame infrared2_optical_frame publish_pointcloud:=true color_ur:=30.0 ir_ur:=30.0 depth_ur:=30.0" >
     <!-- Load parameters to model's main link-->
     <xacro:property name="deg_to_rad" value="0.01745329251994329577" />
@@ -42,5 +42,5 @@
         </camera>
         <always_on>1</always_on>
-        <update_rate>30</update_rate>
+        <update_rate>${color_ur}</update_rate>
         <visualize>1</visualize>
       </sensor>
@@ -64,5 +64,5 @@
         </camera>
         <always_on>1</always_on>
-        <update_rate>90</update_rate>
+        <update_rate>${ir_ur}</update_rate>
         <visualize>0</visualize>
       </sensor>
@@ -86,5 +86,5 @@
         </camera>
         <always_on>1</always_on>
-        <update_rate>90</update_rate>
+        <update_rate>${ir_ur}</update_rate>
         <visualize>0</visualize>
       </sensor>
@@ -107,5 +107,5 @@
         </camera>
         <always_on>1</always_on>
-        <update_rate>90</update_rate>
+        <update_rate>${depth_ur}</update_rate>
         <visualize>0</visualize>
       </sensor>
@@ -114,7 +114,7 @@
       <plugin name="${topics_ns}" filename="librealsense_gazebo_plugin.so">
         <prefix>${camera_name}</prefix>
-        <depthUpdateRate>30.0</depthUpdateRate>
-        <colorUpdateRate>30.0</colorUpdateRate>
-        <infraredUpdateRate>30.0</infraredUpdateRate>
+        <depthUpdateRate>${depth_ur}</depthUpdateRate>
+        <colorUpdateRate>${color_ur}</colorUpdateRate>
+        <infraredUpdateRate>${ir_ur}</infraredUpdateRate>
         <depthTopicName>depth/image_raw</depthTopicName>
         <depthCameraInfoTopicName>depth/camera_info</depthCameraInfoTopicName>
