Commit message: add camera rate parameters

File: urdf/_d435.urdf.xacro (robot description, xacro)
@@ -9,5 +9,5 @@
   <!--File includes-->
   <xacro:include filename="$(find realsense2_description)/urdf/_d435.gazebo.xacro"/>
-  <xacro:macro name="sensor_d435" params="name:=camera topics_ns:=camera parent *origin publish_pointcloud:=true">
+  <xacro:macro name="sensor_d435" params="name:=camera topics_ns:=camera parent *origin publish_pointcloud:=true color_ur:=30.0 ir_ur:=30.0 depth_ur:=30.0">
     <xacro:property name="M_PI" value="3.1415926535897931" />
     <!-- The following values are approximate, and the camera node
@@ -119,5 +119,17 @@
     <link name="${name}_color_optical_frame"/>
     <!-- Realsense Gazebo Plugin -->
-    <xacro:gazebo_d435 camera_name="${name}" reference_link="${name}_link" topics_ns="${topics_ns}" depth_optical_frame="${name}_depth_optical_frame" color_optical_frame="${name}_color_optical_frame" infrared1_optical_frame="${name}_left_ir_optical_frame" infrared2_optical_frame="${name}_right_ir_optical_frame" publish_pointcloud="${publish_pointcloud}"/>
+    <xacro:gazebo_d435
+        camera_name="${name}"
+        reference_link="${name}_link"
+        topics_ns="${topics_ns}"
+        depth_optical_frame="${name}_depth_optical_frame"
+        color_optical_frame="${name}_color_optical_frame"
+        infrared1_optical_frame="${name}_left_ir_optical_frame"
+        infrared2_optical_frame="${name}_right_ir_optical_frame"
+        publish_pointcloud="${publish_pointcloud}"
+        color_ur="${color_ur}"
+        ir_ur="${ir_ur}"
+        depth_ur="${depth_ur}"
+    />
   </xacro:macro>
 </robot>
